File: PCB/MuscleRoller.kicad_pcb (KiCad board)
At the start: 2 copper layers, 83 x 71 mm, 52 parts, among them J1 Conn_01x06_Male, J10 Conn_01x06_Male, J11 Conn_01x06_Male, J12 Conn_01x06_Male, J13 Conn_02x03_Odd_Even, J14 Conn_02x03_Odd_Even, J15 Conn_02x03_Odd_Even, J16 Conn_01x04_Male, J17 Conn_01x04_Male, J18 Conn_01x04_Male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

Commit message: PCB complete
Parts:
- removed A3, A4, A5: Pololu_Breakout_DRV8825, Module:Pololu_Breakout-16_15.2x20.3mm
- removed C10: 0.1U, Capacitor_SMD:C_0805_2012Metric_Pad1.18x1.45mm_HandSolder
- removed C11: 100U, Capacitor_SMD:CP_Elec_6.3x7.7
- removed C12, C13, C14: 100u, Capacitor_SMD:CP_Elec_6.3x7.7
- removed C15, C16, C17, C7, C8: 0.1u, Capacitor_SMD:C_0805_2012Metric_Pad1.18x1.45mm_HandSolder
- removed C9: 1U, Capacitor_SMD:C_0805_2012Metric_Pad1.18x1.45mm_HandSolder
- removed J13, J14, J15: Conn_02x03_Odd_Even, Connector_PinHeader_2.54mm:PinHeader_2x03_P2.54mm_Vertical
- removed J16, J17, J18, J19: Conn_01x04_Male, Connector_JST:JST_XH_B4B-XH-A_1x04_P2.50mm_Vertical
- removed R5: 0.1, Resistor_SMD:R_0805_2012Metric_Pad1.20x1.40mm_HandSolder
- removed U3: ZXBM5210-S, Package_SO:SOIC-8_3.9x4.9mm_P1.27mm
- removed U4: TB67H451FNG,EL, Package_SO:SOIC-8-1EP_3.9x4.9mm_P1.27mm_EP2.29x3mm_ThermalVias
- J1: value Conn_01x06_Male -> Screw_Terminal_01x02; footprint Connector_JST:JST_XH_B6B-XH-A_1x06_P2.50mm_Vertical -> TerminalBlock_Phoenix:TerminalBlock_Phoenix_MKDS-1,5-2_1x02_P5.00mm_Horizontal
- J10: value Conn_01x06_Male -> Conn_01x04_Male; footprint Connector_JST:JST_XH_B6B-XH-A_1x06_P2.50mm_Vertical -> Connector_JST:JST_XH_B4B-XH-A_1x04_P2.50mm_Vertical
- J11, J12: value Conn_01x06_Male -> Conn_01x03_Male; footprint Connector_JST:JST_XH_B6B-XH-A_1x06_P2.50mm_Vertical -> Connector_JST:JST_XH_B3B-XH-A_1x03_P2.50mm_Vertical
- J2: value Conn_01x06_Male -> Conn_02x03_Odd_Even; footprint Connector_JST:JST_XH_B6B-XH-A_1x06_P2.50mm_Vertical -> Connector_PinHeader_2.54mm:PinHeader_2x03_P2.54mm_Vertical
- J3: value Screw_Terminal_01x02 -> Conn_02x03_Odd_Even; footprint TerminalBlock_Phoenix:TerminalBlock_Phoenix_MKDS-1,5-2_1x02_P5.00mm_Horizontal -> Connector_PinHeader_2.54mm:PinHeader_2x03_P2.54mm_Vertical
- J4, J5: value Conn_02x03_Odd_Even -> Conn_01x04_Male; footprint Connector_PinHeader_2.54mm:PinHeader_2x03_P2.54mm_Vertical -> Connector_JST:JST_XH_B4B-XH-A_1x04_P2.50mm_Vertical
- J9: value Conn_01x02_Male -> Conn_01x04_Male; footprint Connector_JST:JST_XH_B2B-XH-A_1x02_P2.50mm_Vertical -> Connector_JST:JST_XH_B4B-XH-A_1x04_P2.50mm_Vertical
- R4: value 47K -> 10K
- moved J9 82.0 mm to (59.5, 103.0), turned to 90 degrees
- moved J10 71.1 mm to (59.5, 85.0), turned to 90 degrees
- moved J1 63.5 mm to (66.5, 62.0), turned to 270 degrees
- moved J2 57.3 mm to (79.8, 96.5), turned to 0 degrees
- moved S2 34.5 mm to (94.0, 55.0)
- moved J5 32.7 mm to (101.5, 97.5), turned to 180 degrees
- moved J11 30.4 mm to (109.0, 105.0), turned to 270 degrees
- moved J4 23.2 mm to (101.5, 105.0), turned to 180 degrees
- moved J12 21.3 mm to (109.0, 93.5), turned to 270 degrees
- moved J3 17.2 mm to (79.8, 73.2), turned to 0 degrees
- moved S1 15.5 mm to (103.5, 55.0)
Connections:
- net DIR1 renamed DIRZ
- net STEP1 renamed STEPZ
- A1 pad 15: STEP0 -> STEPX
- A1 pad 16: DIR0 -> DIRX
- A1 pad 3: Net-(A1-Pad3) -> XA2
- A1 pad 4: Net-(A1-Pad4) -> XA1
- A1 pad 5: Net-(A1-Pad5) -> XB1
- A1 pad 6: Net-(A1-Pad6) -> XB2
- A1 pad 9: EN0 -> ENX
- A2 pad 3: Net-(A2-Pad3) -> ZA2
- A2 pad 4: Net-(A2-Pad4) -> ZA1
- A2 pad 5: Net-(A2-Pad5) -> ZB1
- A2 pad 6: Net-(A2-Pad6) -> ZB2
- A2 pad 9: EN1 -> ENZ
- J1 pad 1: +3V3 -> +12V
- J10 pad 1: +3V3 -> ZB2
- J10 pad 2: GND -> ZB1
- J10 pad 3: CLK -> ZA2
- J10 pad 4: MISO -> ZA1
- J11 pad 3: CLK -> HOMX
- J12 pad 3: CLK -> HOMZ
- J2 pad 2: GND -> Net-(A1-Pad12)
- J2 pad 3: CLK -> +3V3
- J2 pad 4: MISO -> Net-(A1-Pad11)
- J2 pad 5: CS1 -> +3V3
- J2 pad 6: MOSI -> Net-(A1-Pad10)
- J3 pad 1: +12V -> +3V3
- J3 pad 2: GND -> Net-(A2-Pad12)
- J4 pad 2: Net-(A1-Pad12) -> GND
- J4 pad 3: +3V3 -> LC_CLK
- J4 pad 4: Net-(A1-Pad11) -> LC_DAT
- J5 pad 2: Net-(A2-Pad12) -> GND
- J5 pad 3: +3V3 -> LC_CLK2
- J5 pad 4: Net-(A2-Pad11) -> LC_DAT2
- J7 pad 1: Net-(A1-Pad6) -> XB2
- J7 pad 2: Net-(A1-Pad5) -> XB1
- J7 pad 3: Net-(A1-Pad4) -> XA1
- J7 pad 4: Net-(A1-Pad3) -> XA2
- J8 pad 1: Net-(A2-Pad6) -> ZB2
- J8 pad 2: Net-(A2-Pad5) -> ZB1
- J8 pad 3: Net-(A2-Pad4) -> ZA1
- J8 pad 4: Net-(A2-Pad3) -> ZA2
- J9 pad 1: OUT2 -> XB2
- J9 pad 2: OUT1 -> XB1
- U2 pad 11: EN3 -> Net-(U2-Pad11)
- U2 pad 12: DIR2 -> ENZ
- U2 pad 13: STEP2 -> CHARGE
- U2 pad 14: EN2 -> DIRX
- U2 pad 15: EN1 -> STEPX
- U2 pad 16: CHARGE -> ENX
- U2 pad 17: DIR0 -> LC_CLK
- U2 pad 18: STEP0 -> LC_DAT
- U2 pad 19: EN0 -> LC_CLK2
- U2 pad 20: DAC1 -> LC_DAT2
- U2 pad 22: STEP3 -> Net-(U2-Pad22)
- U2 pad 23: DIR3 -> Net-(U2-Pad23)
- U2 pad 24: EN4 -> Net-(U2-Pad24)
- U2 pad 25: STEP4 -> Net-(U2-Pad25)
- U2 pad 27: DIR4 -> HOMZ
- U2 pad 28: CS4 -> HOMX
- U2 pad 29: CLK -> Net-(U2-Pad29)
- U2 pad 30: CS3 -> Net-(U2-Pad30)
- U2 pad 31: MOSI -> Net-(U2-Pad31)
- U2 pad 32: MOT1 -> Net-(U2-Pad32)
- U2 pad 33: MOT2 -> Net-(U2-Pad33)
- U2 pad 34: MISO -> Net-(U2-Pad34)
- U2 pad 35: CS2 -> Net-(U2-Pad35)
- U2 pad 36: CS1 -> Net-(U2-Pad36)
- U2 pad 39: CS0 -> Net-(U2-Pad39)
- U2 pad 6: LC_CLK -> Net-(U2-Pad6)
- U2 pad 7: LC_DAT -> Net-(U2-Pad7)
Routing:
- net +12V: track 230.2 -> 118.4 mm
- net DAC1: track 66.4 -> 0.00 mm, vias 2 -> 0
- net EN4: track 59.9 -> 0.00 mm
- net EN3: track 53.6 -> 0.00 mm, vias 1 -> 0
- net CLK: track 46.8 -> 0.00 mm
- net MOT2: track 46.5 -> 0.00 mm, vias 2 -> 0
- net MISO: track 44.6 -> 0.00 mm
- net STEP4: track 43.0 -> 0.00 mm
- net MOT1: track 41.3 -> 0.00 mm, vias 2 -> 0
- net MOSI: track 38.5 -> 0.00 mm
- net DIR4: track 37.8 -> 0.00 mm
- net EN2: track 35.6 -> 0.00 mm, vias 1 -> 0
- net IO0: track 44.6 -> 15.2 mm
- net STEP3: track 28.7 -> 0.00 mm
- net EN0: track 27.3 -> 0.00 mm
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Other:
- board size 83 x 71 mm -> 66 x 64 mm
- board text added: "3V3"
- board text added: "HOMX"
- board text added: "HOMZ"
- board text added: "XL"
- board text added: "XR"
- board text added: "ZL"
- board text added: "ZR"
- board text removed: "+"
- board text removed: "0"
- board text removed: "1"
- board text removed: "2"
- board text removed: "3"
- board text removed: "4"
- board text removed: "G"
- board text removed: "SAGE ROBOTS A4 2.0"

Commit message: PCB order
Connections:
- J10 pad 3: ZA2 -> ZA1
- J10 pad 4: ZA1 -> ZA2
- J9 pad 3: XA2 -> XA1
- J9 pad 4: XA1 -> XA2
Routing:
- net ZA2: track 15.2 -> 14.2 mm
- net ZA1: track 15.2 -> 14.2 mm
- net XA2: track 17.0 -> 16.0 mm
- net XA1: track 17.0 -> 16.0 mm

Commit message: PCB complete
Parts:
- removed J12: Conn_01x03_Male, Connector_JST:JST_XH_B3B-XH-A_1x03_P2.50mm_Vertical
- added R5: 10K, Resistor_SMD:R_0805_2012Metric_Pad1.20x1.40mm_HandSolder, F.Cu at (165.0, 94.5)
- C2: value 22u -> 100u; footprint Capacitor_SMD:C_0805_2012Metric_Pad1.18x1.45mm_HandSolder -> Capacitor_SMD:CP_Elec_6.3x7.7
- C4: value 100u -> 1u; footprint Capacitor_SMD:CP_Elec_6.3x7.7 -> Capacitor_SMD:C_0805_2012Metric_Pad1.18x1.45mm_HandSolder
- C5: value 0.1u -> 22U
- C6: value 1u -> 0.1u
- J1: value Screw_Terminal_01x02 -> Conn_01x06_Male; footprint TerminalBlock_Phoenix:TerminalBlock_Phoenix_MKDS-1,5-2_1x02_P5.00mm_Horizontal -> Connector_JST:JST_XH_B6B-XH-A_1x06_P2.50mm_Vertical
- J10: value Conn_01x04_Male -> Conn_01x03_Male; footprint Connector_JST:JST_XH_B4B-XH-A_1x04_P2.50mm_Vertical -> Connector_JST:JST_XH_B3B-XH-A_1x03_P2.50mm_Vertical
- J2: value Conn_02x03_Odd_Even -> Conn_01x06_Male; footprint Connector_PinHeader_2.54mm:PinHeader_2x03_P2.54mm_Vertical -> Connector_JST:JST_XH_B6B-XH-A_1x06_P2.50mm_Vertical
- J3: value Conn_02x03_Odd_Even -> Screw_Terminal_01x02; footprint Connector_PinHeader_2.54mm:PinHeader_2x03_P2.54mm_Vertical -> TerminalBlock_Phoenix:TerminalBlock_Phoenix_MKDS-1,5-2_1x02_P5.00mm_Horizontal
- J9: value Conn_01x04_Male -> Screw_Terminal_01x02; footprint Connector_JST:JST_XH_B4B-XH-A_1x04_P2.50mm_Vertical -> TerminalBlock_Phoenix:TerminalBlock_Phoenix_MKDS-1,5-2_1x02_P5.00mm_Horizontal
- R3: value 10K -> 47k
- U2: value ESP32-S2-WROOM -> ESP32-WROOM-E; footprint A4:ESP32-S2-WROOM -> Espressif:ESP32-WROOM-32E
- moved J1 110.3 mm to (159.0, 122.0), turned to 0 degrees
- moved J10 107.3 mm to (164.5, 107.0), turned to 0 degrees
- moved S2 89.2 mm to (171.0, 100.0)
- moved J2 85.7 mm to (159.0, 129.0)
- moved S1 78.0 mm to (171.0, 94.0)
- moved A2 72.5 mm to (123.0, 125.0)
- moved J8 67.7 mm to (111.5, 136.0)
- moved C2 66.2 mm to (129.2, 119.0), turned to 0 degrees
- moved R3 63.8 mm to (153.0, 114.5), turned to 0 degrees
- moved R4 61.6 mm to (156.5, 114.5), turned to 0 degrees
- moved C5 59.9 mm to (139.0, 94.5)
- moved C4 59.7 mm to (138.0, 97.5), turned to 180 degrees
- moved J6 58.8 mm to (162.5, 99.5), turned to 180 degrees
- moved C3 58.8 mm to (129.5, 140.5), turned to 0 degrees
- moved U2 58.2 mm to (149.7, 101.7)
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Connections:
- A1 pad 12: Net-(A1-Pad12) -> MSX
- A1 pad 8: +12V -> ESTOP12V
- A1 pad 9: ENX -> EN_STEP
- A2 pad 12: Net-(A2-Pad12) -> MSZ
- A2 pad 8: +12V -> ESTOP12V
- A2 pad 9: ENZ -> EN_STEP
- C2 pad 1: +3V3 -> ESTOP12V
- C3 pad 1: +12V -> ESTOP12V
- C4 pad 1: +12V -> EN
- C6 pad 1: EN -> +3V3
- J1 pad 1: +12V -> +3V3
- J10 pad 1: ZB2 -> +3V3
- J10 pad 2: ZB1 -> GND
- J10 pad 3: ZA1 -> HOMX
- J11 pad 3: HOMX -> HOMZ
- J2 pad 2: Net-(A1-Pad12) -> GND
- J2 pad 3: +3V3 -> CLK
- J2 pad 4: Net-(A1-Pad11) -> MISO
- J2 pad 5: +3V3 -> CS1
- J2 pad 6: Net-(A1-Pad10) -> MOSI
- J3 pad 1: +3V3 -> +12V
- J3 pad 2: Net-(A2-Pad12) -> GND
- J9 pad 1: XB2 -> +12V
- J9 pad 2: XB1 -> ESTOP12V
- R3 pad 1: +3V3 -> ESTOP12V
- R3 pad 2: EN -> ESTOP
- R4 pad 1: +3V3 -> ESTOP
- R4 pad 2: DAC2 -> GND
- U2 pad 10: Net-(U2-Pad10) -> STEPZ
- U2 pad 11: Net-(U2-Pad11) -> MSZ
- U2 pad 12: ENZ -> LC_CLK
- U2 pad 13: CHARGE -> LC_DAT
- U2 pad 14: DIRX -> LC_CLK2
- U2 pad 15: STEPX -> GND
- U2 pad 16: ENX -> LC_DAT2
- U2 pad 17: LC_CLK -> Net-(U2-Pad17)
- U2 pad 18: LC_DAT -> Net-(U2-Pad18)
- U2 pad 19: LC_CLK2 -> Net-(U2-Pad19)
- U2 pad 20: LC_DAT2 -> Net-(U2-Pad20)
- U2 pad 21: DAC2 -> Net-(U2-Pad21)
- U2 pad 23: Net-(U2-Pad23) -> ESTOP
- U2 pad 25: Net-(U2-Pad25) -> IO0
- U2 pad 26: GND -> CLK
- U2 pad 27: HOMZ -> MISO
- U2 pad 28: HOMX -> CS0
- U2 pad 29: Net-(U2-Pad29) -> MOSI
- U2 pad 3: IO0 -> EN
- U2 pad 30: Net-(U2-Pad30) -> CS1
- U2 pad 31: Net-(U2-Pad31) -> HOMZ
- U2 pad 33: Net-(U2-Pad33) -> HOMX
- U2 pad 34: Net-(U2-Pad34) -> TX
- U2 pad 35: Net-(U2-Pad35) -> RX
- U2 pad 37: RX -> Net-(U2-Pad37)
- U2 pad 38: TX -> GND
- U2 pad 39: Net-(U2-Pad39) -> (no net)
- U2 pad 4: DIRZ -> CHARGE
- U2 pad 5: STEPZ -> DIRX
- U2 pad 6: Net-(U2-Pad6) -> STEPX
- U2 pad 7: Net-(U2-Pad7) -> MSX
- U2 pad 8: Net-(U2-Pad8) -> EN_STEP
- U2 pad 9: Net-(U2-Pad9) -> DIRZ
Routing:
- net ESTOP12V: track 0.00 -> 101.5 mm
- net +12V: track 118.4 -> 44.9 mm
- net GND: track 187.4 -> 140.1 mm
- net EN_STEP: track 0.00 -> 42.5 mm
- net CS1: track 0.00 -> 39.8 mm
- net MOSI: track 0.00 -> 32.0 mm
- net MSZ: track 0.00 -> 30.1 mm
- net ENX: track 26.0 -> 0.00 mm
- net MISO: track 0.00 -> 25.5 mm
- net CS0: track 0.00 -> 22.0 mm
- net CLK: track 0.00 -> 22.0 mm
- net STEPZ: track 4.57 -> 23.8 mm
- net DIRZ: track 4.14 -> 22.6 mm
- net +3V3: track 16.6 -> 34.3 mm, vias 1 -> 4
- net MSX: track 0.00 -> 14.0 mm
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Other:
- board size 66 x 64 mm -> 70 x 70 mm
- board text added: "G R T"
- board text added: "LC2"
- board text added: "SPI Z"
- board text added: "X"
- board text added: "Z"
- board text removed: "3V3"
- board text removed: "GND"
- board text removed: "IO0"
- board text removed: "LC_DAT"
- board text removed: "RX"
- board text removed: "TX"
- board text removed: "XL"
- board text removed: "XR"
- board text removed: "ZL"
- board text removed: "ZR"
